File: Documentation/Circuit Diagrams/Display.sch (EAGLE design)
At the start: 37 parts, among them IC1 CY62256LL-SNC, IC10 4053D, IC13 4001D, IC15 4081D, IC16 4053D, IC17 4053D, IC18 4053D, IC19 4053D, IC20 4053D, IC21 4053D, IC22 4053D, IC23 4053D, IC3 4053D, IC8 4081D, IC9 4027D

Commit message: Fixed some logical flow errors
Parts:
- removed IC1: CY62256LL-SNC, memory-sram:CY62256LL-SNC
- removed IC3: 4053D, 40xx:4053D
- added MUX_ADDRESS: 4053D, 40xx:4053D
- added RAM_FIELD: CY62256LL-SNC, memory-sram:CY62256LL-SNC
- renumbered IC19 to SHIFT_DOWN_MUX, IC23 to REWRITE_MUX
Connections:
- removed net FF_READ/WRITE: FF_R/W(H=WRITE)A.Q, IC20A.INH, IC21A.INH, IC22A.INH, REWRITE_MUXA.INH
- removed net N$41: IC10A.A, IC10A.B, IC10A.C
- removed net N$44: FF_R/W(H=WRITE)A.!Q, IC1G$1.!WE
- new net !FF_READ/WRITE: FF_R/W(H=WRITE)A.!Q, IC20A.INH, IC21A.INH, IC22A.INH, RAM_FIELDG$1.!WE, REWRITE_MUXA.INH
- new net N$14: FF_R/W(H=WRITE)A.Q, IC10A.A, IC10A.B, IC10A.C, MUX_ADDRESSA.A, MUX_ADDRESSA.B, MUX_ADDRESSA.C
- net N$15: now also RAM_FIELDG$1.DQ5; no longer IC1G$1.DQ5
- net N$20: now also MUX_ADDRESSA.Y0; no longer IC3A.Y0, OVERLAPLOGIC.I1
- net N$21: now also RAM_FIELDG$1.DQ3; no longer IC1G$1.DQ3
- net N$23: now also MUX_ADDRESSA.X0; no longer IC3A.X0, OVERLAPLOGIC.CLK
- net N$24: now also RAM_FIELDG$1.DQ7; no longer IC1G$1.DQ7
- net N$25: now also MUX_ADDRESSA.X1; no longer IC3A.X1
- net N$26: no longer OVERLAPLOGIC.I3
- net N$27: now also MUX_ADDRESSA.Y1, OVERLAPLOGIC.I1; no longer IC3A.Y1
- net N$36: now also OVERLAPLOGIC.I2
- net N$37: now also OVERLAPLOGIC.I3
- net N$38: now also MUX_ADDRESSA.X, RAM_FIELDG$1.A11; no longer IC1G$1.A11, IC3A.X
- net N$39: now also MUX_ADDRESSA.Y, RAM_FIELDG$1.A12; no longer IC1G$1.A12, IC3A.Y
- net N$40: now also OVERLAPLOGIC.CLK; no longer IC3A.A, IC3A.B, IC3A.C
- net N$42: now also RAM_FIELDG$1.A13; no longer IC1G$1.A13
- net N$43: now also RAM_FIELDG$1.A14; no longer IC1G$1.A14
- net N$45: now also RAM_FIELDG$1.DQ2; no longer IC1G$1.DQ2
- net N$46: now also RAM_FIELDG$1.DQ1; no longer IC1G$1.DQ1
- net N$47: now also RAM_FIELDG$1.DQ4; no longer IC1G$1.DQ4
- net N$51: now also RAM_FIELDG$1.DQ0; no longer IC1G$1.DQ0
- net N$57: now also RAM_FIELDG$1.DQ6; no longer IC1G$1.DQ6
- net N$9: no longer OVERLAPLOGIC.I2
- net PE: now also MUX_ADDRESSA.INH, RAM_FIELDG$1.!CE, RAM_FIELDG$1.!OE, RAM_FIELDG$1.A0, RAM_FIELDG$1.A1, RAM_FIELDG$1.A10, RAM_FIELDG$1.A2, RAM_FIELDG$1.A3, RAM_FIELDG$1.A4, RAM_FIELDG$1.A5, RAM_FIELDG$1.A6, RAM_FIELDG$1.A7, RAM_FIELDG$1.A8, RAM_FIELDG$1.A9; no longer IC1G$1.!CE, IC1G$1.!OE, IC1G$1.A0, IC1G$1.A1, IC1G$1.A10, IC1G$1.A2, IC1G$1.A3, IC1G$1.A4, IC1G$1.A5, IC1G$1.A6, IC1G$1.A7, IC1G$1.A8, IC1G$1.A9, IC3A.INH
Other:
- moved on the sheet: STATE

Commit message: Update
Parts:
- added DISPLAY_SINK: 4514N, 45xx:4514N
- added FULL/RESET, IC1, IC3, RESETBUTTONOR!COLLISION: 4071D, 40xx:4071D
- added R1: (no value), rcl:R-US_0204/7
- added RESETEVERYTHING: (no value), switch:REKN
- renumbered REWRITE_MUX to WRITESELECT
Connections:
- removed net N$25: MUX_ADDRESSA.X1, STATEA.Q0
- removed net N$26: IC10A.Y0, RAMADDRESSA.Q1, STATEA.P3
- removed net N$37: IC10A.Y1, OVERLAPLOGIC.I3, STATEA.Q3
- removed net N$51: RAM_FIELDG$1.DQ0, SR_ONE_1A.P0, SR_TWO_1A.P0, WRITESELECTA.X
- removed net N$62: 8INANDOR.I7, IC16A.Y0, SR_TWO_2A.Q3
- removed net N$67: SHIFT_DOWN_MUXA.X1, SR_ONE_1A.Q0
- removed net N$74: IC16A.Y1, SR_ONE_2A.Q3
- removed net N$78: IC16A.Y, SR_FOUR_2A.P3
- removed net N$79: SHIFT_DOWN_MUXA.X, SR_FOUR_1A.P0
- removed net N$81: OR_DISPLAY_1B.I1, SR_FOUR_1A.Q0, WRITESELECTA.X0
- removed net N$88: IC20A.Y0, OR_DISPLAY_2A.I0, SR_FOUR_2A.Q3
- removed net N$90: OR_DISPLAY_1B.O, WRITESELECTA.X1
- removed net N$97: IC20A.Y1, OR_DISPLAY_2A.O
- new net !COLLISION: RESETBUTTONOR!COLLISIONA.I0
- new net ADD_LSB: DISPLAY_SINKA.D1, IC10A.Y0, IC10A.Y1, OVERLAPLOGIC.I3, OVERLAPLOGIC.I7, RAMADDRESSA.Q1, ROWBOTTOMA.Q1, STATEA.P3, STATEA.Q3
- new net ADD_MSB: DISPLAY_SINKA.D4, IC8A.I0, MUX_ADDRESSA.X0, MUX_ADDRESSA.X1, OVERLAPLOGIC.I4, RAMADDRESSA.Q4, ROWBOTTOMA.Q4, STATEA.P0, STATEA.Q0
- new net LEASTSIG: OR_DISPLAY_2A.I1
- new net MOSTSIG: OR_DISPLAY_1B.I0
- new net RESETBUTTON: FULL/RESETA.I0, IC1A.I1, RAMADDRESSA.PE, RESETBUTTONOR!COLLISIONA.I1, RESETEVERYTHING.1@B, SR_FOUR_1A.RES, SR_FOUR_2A.RES, SR_ONE_1A.RES, SR_ONE_2A.RES
- net !FF_READ/WRITE: now also IC1A.I0; no longer IC20A.INH, IC21A.INH, IC22A.INH, WRITESELECTA.INH
- net FULL_ROW: now also 8INANDOR.AND, FULL/RESETA.I1; no longer 8INANDOR.O1, SR_TWO_1A.RES, SR_TWO_2A.RES
- net LSB: now also 8INANDOR.CLK, OR_DISPLAY_1B.I1, OR_DISPLAY_1B.O, RAM_FIELDG$1.DQ0, SHIFT_DOWN_MUXA.X, SHIFT_DOWN_MUXA.X0, SHIFT_DOWN_MUXA.X1, SR_FOUR_1A.P0, SR_FOUR_1A.Q0, SR_ONE_1A.P0, SR_ONE_1A.Q0, SR_TWO_1A.P0, SR_TWO_1A.Q0, WRITESELECTA.X, WRITESELECTA.X0, WRITESELECTA.X1; no longer OR_DISPLAY_2A.I1
- net MSB: now also 8INANDOR.I7, IC16A.Y, IC16A.Y0, IC16A.Y1, IC20A.Y, IC20A.Y0, IC20A.Y1, OR_DISPLAY_2A.I0, OR_DISPLAY_2A.O, RAM_FIELDG$1.DQ7, SR_FOUR_2A.P3, SR_FOUR_2A.Q3, SR_ONE_2A.P3, SR_ONE_2A.Q3, SR_TWO_2A.P3, SR_TWO_2A.Q3; no longer OR_DISPLAY_1B.I0
- net N$2: now also IC1A.O, IC20A.INH, IC21A.INH, IC22A.INH, WRITESELECTA.INH; no longer IC8A.I0, OVERLAPLOGIC.I4, ROWBOTTOMA.Q4
- net N$23: now also FULL/RESETA.O, SR_TWO_1A.RES, SR_TWO_2A.RES; no longer MUX_ADDRESSA.X0, RAMADDRESSA.Q4, STATEA.P0
- net N$24: now also IC3A.I0, IC8A.O; no longer IC20A.Y, RAM_FIELDG$1.DQ7, SR_ONE_2A.P3, SR_TWO_2A.P3
- net N$27: now also DISPLAY_SINKA.D3
- net N$36: now also DISPLAY_SINKA.D2
- net N$5: now also IC3A.O; no longer IC8A.O
- net N$6: now also IC3A.I1, RESETBUTTONOR!COLLISIONA.O; no longer OVERLAPLOGIC.I7, ROWBOTTOMA.Q1
- net N$64: now also 8INANDOR.OR; no longer 8INANDOR.O2
- net N$8: now also R1.1, RESETEVERYTHING.1@A; no longer 8INANDOR.CLK, SHIFT_DOWN_MUXA.X0, SR_TWO_1A.Q0
- net PE: now also DISPLAY_SINKA.INH, R1.2; no longer RAMADDRESSA.PE, SR_FOUR_1A.RES, SR_FOUR_2A.RES, SR_ONE_1A.RES, SR_ONE_2A.RES
- net V+: now also DISPLAY_SINKA.ST, RESETEVERYTHING.0@A
Other:
- moved on the sheet: ROWBOTTOM
